File: Hardware/FitnessTracker.sch (KiCad schematic (older format))
At the start: 60 parts, among them IC1 MAX30102, J1 ST_Link, Q1 BSS138, Q2 BSS138, Q3 BSS138, U1 STM32WB15CCU6E, U2 LIS2DS12TR, U3 MS560702BA03-50, U4 ublox_SAM-M8Q, Y1 32.768kHz, Y2 32MHz

Commit message: schematic complete, begining pcb layout process
Parts:
- AE1: footprint MLPF-WB55-01E3_STM -> footprints:MLPF-WB55-01E3
- AE2: footprint (none) -> footprints:2.4GHz Antenna
- BT1: footprint (none) -> Connector_PinHeader_2.54mm:PinHeader_1x02_P2.54mm_Vertical
- C1, C10, C11, C12, C13, C14, C15, C16, C17, C18, C19, C2, C20, C21, C22, C3, C4, C5, C6, C7, C8, C9: footprint (none) -> Capacitor_SMD:C_0402_1005Metric
- C23, C24, C25, C26, C27, C28: renamed from C?; footprint (none) -> Capacitor_SMD:C_0402_1005Metric
- J1: footprint (none) -> Connector_PinHeader_2.54mm:PinHeader_1x05_P2.54mm_Vertical
- J2: renamed from J?; footprint (none) -> Connector_PinHeader_2.54mm:PinHeader_1x04_P2.54mm_Vertical
- L1: footprint (none) -> Inductor_SMD:L_0402_1005Metric
- L2: renamed from L?; footprint (none) -> Inductor_SMD:L_0402_1005Metric
- R1, R10, R11, R12, R2, R3, R4, R5, R6, R7, R8, R9: footprint (none) -> Resistor_SMD:R_0402_1005Metric
- TP1: footprint (none) -> TestPoint:TestPoint_Pad_1.0x1.0mm
- U6: renamed from U?; footprint SOT_020C18R_STM -> footprints:STLQ020C18R
- Y1, Y2: footprint (none) -> footprints:8Q20000MAAVT
- gave numbers to parts that had none: 1
Connections:
- wire segments 106 -> 105
Other:
- moved on the sheet: U1, Y2

Commit message: completed rough layout of pcb
Parts:
- removed C19: 100nF, Capacitor_SMD:C_0402_1005Metric, symbol Device:C_Small
- removed J1: ST_Link, Connector_PinHeader_2.54mm:PinHeader_1x05_P2.54mm_Vertical, symbol Connector_Generic:Conn_01x05
- removed J2: SAM_UART, Connector_PinHeader_2.54mm:PinHeader_1x04_P2.54mm_Vertical, symbol Connector_Generic:Conn_01x04
- removed Q1: BSS138, Package_TO_SOT_SMD:SOT-23, symbol Transistor_FET:BSS138
- removed R3, R4: 1M, Resistor_SMD:R_0402_1005Metric, symbol Device:R_Small
- added J1: PWR_OUT, Connector_PinHeader_1.00mm:PinHeader_1x02_P1.00mm_Vertical, symbol Connector_Generic:Conn_01x02
- added J2: GPS_UART, Connector_PinHeader_1.00mm:PinHeader_1x02_P1.00mm_Vertical, symbol Connector_Generic:Conn_01x02
- added J3: STLINK, Connector_PinHeader_1.00mm:PinHeader_1x04_P1.00mm_Vertical, symbol Connector_Generic:Conn_01x04
- added J4: LPUART, Connector_PinHeader_1.00mm:PinHeader_1x02_P1.00mm_Vertical, symbol Connector_Generic:Conn_01x02
- added J5: GPIO, Connector_PinHeader_1.00mm:PinHeader_1x03_P1.00mm_Vertical, symbol Connector_Generic:Conn_01x03
- added JP1: BOOT, Jumper:SolderJumper-2_P1.3mm_Open_Pad1.0x1.5mm, symbol Jumper:SolderJumper_2_Open
- AE1: DIGIKEY (none) -> ‎497-19088-1-ND‎
- AE2, BT1, C1, C10, C11, C12, C13, C14, C15, C16, C17, C18, C2, C20, C21, C22, C23, C24, C25, C26, C27, C28, C3, C4, C5, C6, C7, C8, C9, TP1: DIGIKEY (none) -> NA
- IC1: DIGIKEY (none) -> MAX30102EFD+-ND
- L1: DIGIKEY (none) -> 490-6571-1-ND
- Q2, Q3: footprint Package_TO_SOT_SMD:SOT-23 -> Package_TO_SOT_SMD:SOT-323_SC-70; DIGIKEY (none) -> BSS138W-FDITR-ND
- R1: DIGIKEY (none) -> CRGCQ0402J10K‎
- R10, R2, R5, R6, R9: DIGIKEY (none) -> 2037-PFR05S-105-FNHTR-ND
- R11, R12: DIGIKEY (none) -> 2019-RK73B1ETTP471JTR-ND
- R7, R8: DIGIKEY (none) -> 10-ERJ-U02J220XTR-ND
- U1: DIGIKEY (none) -> STM32WB15CCU6E‎
- U2: DIGIKEY (none) -> 497-16261-2-ND
- U3: DIGIKEY (none) -> 223-1198-2-ND
- U4: DIGIKEY (none) -> SAM-M8Q-0-10‎
- U6: DIGIKEY (none) -> STLQ020C18R‎
- Y2: DIGIKEY (none) -> 887-8Q-32.000MEIE-TTR-ND
Connections:
- net +1V8: now also J1.1 (Pin_1), JP1.1 (A)
- net GND: now also R1.2, J1.2 (Pin_2); no longer R1.1
- net NRST: now also J3.4 (Pin_4)
- net SPI_MISO: now also U1.16 (PA6); no longer U1.44 (PB4)
- net SPI_MOSI: now also U1.15 (PA5); no longer U1.45 (PB5)
- net SPI_SCK: now also U1.10 (PA1); no longer U1.43 (PB3)
- net SWCLK: now also J3.2 (Pin_2)
- net SWDIO: now also J3.1 (Pin_1)
- net LPUART_TX: now reaches U1.11 (PA2)
- net LPUART_TX: now also J4.2 (Pin_2)
- net LPUART_RX: now reaches U1.12 (PA3)
- net LPUART_RX: now also J4.1 (Pin_1)
- net ACC_CS: now reaches U1.17 (PA7)
- net ACC_CS: now also U2.2 (CS)
- net BAR_CS: now reaches U1.18 (PA8)
- net BAR_CS: now also U3.4 (SCB)
- net PB0: now reaches U1.28 (PB0)
- net PB0: now also J5.1 (Pin_1)
- net PB1: now reaches U1.29 (PB1)
- net PB1: now also J5.2 (Pin_2)
- net PB13: now reaches U1.30 (PB13)
- net PB13: now also J5.3 (Pin_3)
- net BOOT0: now reaches U1.4 (PH3-BOOT0)
- net BOOT0: now also R1.1, JP1.2 (B); no longer R1.2
- net 30102_INT renamed HRM_INT
- net LIS_INT1 renamed ACC_INT1
- net LIS_INT2 renamed ACC_INT2
- net SAM_INT renamed GPS_INT
- net SAM_INT_LV renamed GPS_INT_LV
- net SAM_RX renamed GPS_RX
- net GPS_RX: now also J2.1 (Pin_1)
- net SAM_TX renamed GPS_TX
- net GPS_TX: now also J2.2 (Pin_2)
- net SPI_NSS1: no longer names the net of U1.20 (PB2)
- net SPI_NSS1: no longer U2.2 (CS)
- net SPI_NSS2: no longer names the net of U1.46 (PB6)
- net SPI_NSS2: no longer U3.4 (SCB)
- new net SWO: J3.3 (Pin_3), U1.43 (PB3)
- no-connect marks 5 -> 20
Other:
- moved on the sheet: C2, C7, C9, R1
